Commit message: upload

File: src/broverette_description/broverette_description/urdf/broverette.urdf (robot description, URDF)
Before this commit: robot broverette, 10 links, 9 joints
Joints:
- joint base_footprint_joint: child base_footprint -> base_link; origin xyz=0 0 0 rpy=0 0 0 -> xyz=0 0 0 rpy=0 0 3.14159; parent base_link -> base_footprint

File: src/broverette_description/urdf/broverette.urdf (robot description, URDF)
Before this commit: robot broverette, 10 links, 9 joints
Links:
- removed link camera_link
Joints:
- removed joint camera_joint
- joint laser_joint: origin xyz=0.049748 -0.0012 0.1165 rpy=0 0 0 -> xyz=0.107 -0.0012 0.0678 rpy=0 0 0
