Commit message: test

File: src/broverette_description/urdf/broverette.urdf (robot description, URDF)
Before this commit: robot broverette, 10 links, 9 joints
Links:
- removed link camera_link
Joints:
- removed joint camera_joint
- joint laser_joint: origin xyz=0.049748 -0.0012 0.1165 rpy=0 0 0 -> xyz=0.049748 -0.0012 0.1165 rpy=3.14159 0 0
